Commit message: fix(isaac): regenerate the URDF the importer actually reads
urdf/vica.urdf still carried the 0.293 m wheel separation that ae3ca96
corrected in VICA.xacro. Isaac's URDF importer takes .urdf, not .xacro, so
the next re-import would have put the old robot back into the stage -- no
error, no warning, and the geometry work silently undone.

Regenerate it, and add export_isaac_urdf.sh so the expansion is a step in
the re-import procedure rather than something remembered:

    1. export_isaac_urdf.sh
    2. Isaac URDF Importer -> urdf/vica.urdf
    3. fixup_vica_usd_joints.py
    4. build_vica_ros_graphs.py

The script checks the result with check_urdf and prints the wheel and laser
origins, the three numbers that have gone wrong before.

Also drop the rear_* caster spellings from fixup_vica_usd_joints.py. The
casters sit behind the drive axle but keep their front_* names to match the
physical robot's package, so accepting both spellings only obscured which
one is real.

Co-Authored-By: Claude Opus 5 (1M context) <noreply@anthropic.com>

File: src/vica_description/urdf/vica.urdf (robot description, URDF)
Before this commit: robot VICA, 11 links, 10 joints
Links:
- link front_left_caster_steer_1: geometry collision box size=0.08 0.08 0.0755; visual mesh filename=package://vica_description/meshes/front_left_caster_steer_1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 scale=0.001 0.001 0.001
- link front_left_caster_wheel_1: geometry collision cylinder length=0.04 radius=0.042; visual mesh filename=package://vica_description/meshes/front_left_caster_wheel_1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 scale=0.001 0.001 0.001
- link front_right_caster_steer_1: geometry collision box size=0.08 0.08 0.0755; visual mesh filename=package://vica_description/meshes/front_right_caster_steer_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 scale=0.001 0.001 0.001
- link front_right_caster_wheel_1: geometry collision cylinder length=0.04 radius=0.042; visual mesh filename=package://vica_description/meshes/front_right_caster_wheel_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 scale=0.001 0.001 0.001
- link laser_frame: geometry visual mesh filename=package://vica_description/meshes/lidar_1.stl scale=0.001 0.001 0.001
Joints:
- joint front_left_caster_steer_joint: origin xyz=-0.222 0.0845 -0.087 rpy=0 0 0 -> xyz=-0.222 0.0845 -0.0825 rpy=0 0 0
- joint front_left_caster_wheel_joint: origin xyz=-0.03 -0.015 -0.0655 rpy=0 0 0 -> xyz=-0.03 -0.005 -0.0655 rpy=0 0 0
- joint front_right_caster_steer_joint: origin xyz=-0.222 -0.0845 -0.087 rpy=0 0 0 -> xyz=-0.222 -0.0845 -0.0825 rpy=0 0 0
- joint front_right_caster_wheel_joint: origin xyz=-0.03 0.015 -0.0655 rpy=0 0 0 -> xyz=-0.03 0.005 -0.0655 rpy=0 0 0
- joint laser_joint: origin xyz=0.185 0.0 0.19 rpy=0 0 0 -> xyz=0.185 0.0 0.192 rpy=0 0 0
- joint left_wheel_joint: origin xyz=0.154 0.1465 -0.125 rpy=0 0 0 -> xyz=0.154 0.182 -0.125 rpy=0 0 0
- joint right_wheel_joint: origin xyz=0.154 -0.1465 -0.125 rpy=0 0 0 -> xyz=0.154 -0.182 -0.125 rpy=0 0 0
