Commit message: feat(urdf): OMX 를 로보티스 실제 메시로 그린다
치수·관절한계·질량은 이미 공식 저장소에서 가져왔지만 메시는 안 가져와서 상자와
원기둥으로 그리고 있었다. 같은 브랜치에 있으므로 가져왔다 — link1..5 와 그리퍼
좌우, meshes/omx/ 에 4 MB.

시각용에만 쓴다. 충돌은 상자로 남는다: 솔버가 시간을 쓰는 것은 콜라이더이고,
움직이는 팔 하나에 링크당 1 MB 짜리 삼각형 더미를 두고 싶은 사람은 없다.

길이를 늘려도 메시는 늘어나지 않는다. 로보티스가 파는 것보다 긴 링크는 우리
부품이고, 그들의 껍데기를 한 축으로 늘려 그리는 것은 존재하지 않는 물건의
그림이다. 실제로 렌더해 보면 팔의 앞쪽 절반이 떨어져 떠 있는 것처럼 보인다 —
관절만 멀어지고 껍데기는 제자리이기 때문이다. 그래서 보여주는 그림은 기본
길이로 만들고, 늘린 값(l3 0.30 / l4 0.28)은 도달거리 계산용 플래그로 남긴다.

export_isaac_urdf.sh 의 VICA_ARM_ARGS 에 기본값을 줬다. set -u 라서 안 넣고
돌리면 "unbound variable" 로 죽었고, 이 스크립트는 인자 없이 돌리는 쪽이
보통이다.

play_stage 는 회전 연산자 종류를 가린다. 팔 테스트룸은 rotateZ(스칼라)를 쓰고
코스는 모두 rotateXYZ(벡터)라, 스폰 각도에 벡터를 쓰던 코드가 팔 스테이지에서만
기동 9초 만에 죽었다:
  Type mismatch for </World/VICA.xformOp:rotateZ>: expected 'float', got 'GfVec3f'

drive_scripted 는 --origin 을 받는다. /odom 은 스폰 지점에서 0 으로 시작하고
replay_render 는 그 좌표를 스테이지 월드로 쓰므로, 스폰이 원점일 때만 둘이
맞는다. 병원과 오피스는 (0,0) 이라 맞았고 팔 테스트룸은 아니었다 — 렌더가 로봇을
꺼내온 좁은 통로에 도로 갖다 놓았다.

Co-Authored-By: Claude Opus 5 (1M context) <noreply@anthropic.com>
Claude-Session: https://claude.ai/code/session_01RnJpDRgBtMFe8arQPicSZr

File: src/vica_description/urdf/omx_arm.xacro (robot description, xacro)
@@ -19,9 +19,12 @@
   drives, including the robot's own, and an include that is missing there
   breaks a file that has nothing to do with arms.
-  The meshes are not in this workspace either. What is drawn below are boxes
-  and cylinders sized from the joint offsets. That is honest about what is
-  known: the kinematics and the masses are ROBOTIS's numbers, the shape is an
-  approximation, and nothing downstream reads the shape except the renderer.
-  Real meshes can be dropped in later without moving a joint.
+  The meshes are ROBOTIS's own, fetched from the same branch into
+  meshes/omx/. They are visual only: collision stays as boxes, because a
+  collider is what the physics solver spends its time on and a 1 MB triangle
+  soup per link is not what anyone wants around a moving arm.
+  Lengthening moves the joints and does not stretch the meshes. A link built
+  longer than ROBOTIS sells is our own part, and drawing their casing scaled
+  along one axis would be a picture of something that does not exist. The mesh
+  sits at the joint and the extra length shows as the gap to the next one.
   Lengthening
   ~~~~~~~~~~~
@@ -63,13 +66,23 @@
     <!-- The arm's own section, for the box stand-ins. -->
     <xacro:property name="w" value="0.045" />
-    <xacro:macro name="omx_link" params="name mass seg axis:=z">
+    <xacro:macro name="omx_link" params="name mass seg axis:=z mesh:=''">
       <link name="${name}">
         <visual>
-          <origin xyz="${axis == 'x' and seg/2 or 0} 0 ${axis == 'z' and seg/2 or 0}"
-                  rpy="0 0 0"/>
-          <geometry>
-            <box size="${axis == 'x' and seg or w} ${w} ${axis == 'z' and seg or w}"/>
-          </geometry>
-          <material name="silver"/>
+          <xacro:if value="${mesh != ''}">
+            <origin xyz="0 0 0" rpy="0 0 0"/>
+            <geometry>
+              <mesh filename="package://vica_description/meshes/omx/${mesh}.stl"
+                    scale="0.001 0.001 0.001"/>
+            </geometry>
+            <material name="silver"/>
+          </xacro:if>
+          <xacro:unless value="${mesh != ''}">
+            <origin xyz="${axis == 'x' and seg/2 or 0} 0 ${axis == 'z' and seg/2 or 0}"
+                    rpy="0 0 0"/>
+            <geometry>
+              <box size="${axis == 'x' and seg or w} ${w} ${axis == 'z' and seg or w}"/>
+            </geometry>
+            <material name="silver"/>
+          </xacro:unless>
         </visual>
         <inertial>
@@ -89,5 +102,5 @@
     </xacro:macro>
     <!-- link1 is the base. Fixed to whatever it is mounted on. -->
-    <xacro:omx_link name="${prefix}link1" mass="${m1}" seg="0.034" axis="z"/>
+    <xacro:omx_link name="${prefix}link1" mass="${m1}" mesh="link1" seg="0.034" axis="z"/>
     <joint name="${prefix}base_joint" type="fixed">
       <xacro:insert_block name="origin"/>
@@ -95,5 +108,5 @@
       <child link="${prefix}link1"/>
     </joint>
-    <xacro:omx_link name="${prefix}link2" mass="${m2}" seg="0.0595" axis="z"/>
+    <xacro:omx_link name="${prefix}link2" mass="${m2}" mesh="link2" seg="0.0595" axis="z"/>
     <joint name="${prefix}joint1" type="revolute">
       <origin xyz="0.012 0.0 0.017" rpy="0 0 0"/>
@@ -104,5 +117,5 @@
              effort="${joint_effort}" velocity="${joint_velocity}"/>
     </joint>
-    <xacro:omx_link name="${prefix}link3" mass="${m3}" seg="${link3_len}" axis="z"/>
+    <xacro:omx_link name="${prefix}link3" mass="${m3}" mesh="link3" seg="${link3_len}" axis="z"/>
     <joint name="${prefix}joint2" type="revolute">
       <origin xyz="0.0 0.0 0.0595" rpy="0 0 0"/>
@@ -113,5 +126,5 @@
              effort="${joint_effort}" velocity="${joint_velocity}"/>
     </joint>
-    <xacro:omx_link name="${prefix}link4" mass="${m4}" seg="${link4_len}" axis="x"/>
+    <xacro:omx_link name="${prefix}link4" mass="${m4}" mesh="link4" seg="${link4_len}" axis="x"/>
     <joint name="${prefix}joint3" type="revolute">
       <!-- 0.024 of forward offset is ROBOTIS's; the vertical part is the
@@ -124,5 +137,5 @@
              effort="${joint_effort}" velocity="${joint_velocity}"/>
     </joint>
-    <xacro:omx_link name="${prefix}link5" mass="${m5}" seg="${link5_len}" axis="x"/>
+    <xacro:omx_link name="${prefix}link5" mass="${m5}" mesh="link5" seg="${link5_len}" axis="x"/>
     <joint name="${prefix}joint4" type="revolute">
       <origin xyz="${link4_len} 0.0 0.0" rpy="0 0 0"/>

File: src/vica_description/urdf/vica_arm.urdf (robot description, URDF)
Before this commit: robot VICA, 25 links, 24 joints
Links:
- link omx_link1: geometry visual mesh filename=package://vica_description/meshes/omx/link1.stl scale=0.001 0.001 0.001
- link omx_link2: geometry visual mesh filename=package://vica_description/meshes/omx/link2.stl scale=0.001 0.001 0.001
- link omx_link3: mass 0.32463086718749995 -> 0.13850917; geometry visual mesh filename=package://vica_description/meshes/omx/link3.stl scale=0.001 0.001 0.001
- link omx_link4: mass 0.29974817419354843 -> 0.13274562; geometry visual mesh filename=package://vica_description/meshes/omx/link4.stl scale=0.001 0.001 0.001
- link omx_link5: geometry visual mesh filename=package://vica_description/meshes/omx/link5.stl scale=0.001 0.001 0.001
Joints:
- joint omx_joint3: origin xyz=0.024 0 0.3 rpy=0 0 0 -> xyz=0.024 0 0.128 rpy=0 0 0
- joint omx_joint4: origin xyz=0.28 0.0 0.0 rpy=0 0 0 -> xyz=0.124 0.0 0.0 rpy=0 0 0
