Commit message: fix(urdf): drop the lidar collision mesh
laser_frame carried lidar_1.stl (124 KB) as a collision geometry. A lidar
has nothing to collide with, and Isaac's URDF importer turns the mesh into
a convex hull that the robot's own RTX scan then reports as an obstacle.

This is the most likely source of the collision_monitor false positive that
forced FootprintApproach to be disabled in vica_nav2_params.yaml. Re-enable
that polygon after confirming a clean run.

The visual mesh is unchanged, so RViz looks identical.

Co-Authored-By: Claude Opus 5 (1M context) <noreply@anthropic.com>

File: src/vica_description/urdf/VICA.xacro (robot description, xacro)
@@ -198,10 +198,6 @@
     <material name="silver"/>
   </visual>
-  <collision>
-    <origin xyz="-0.185 -0.0 -0.258" rpy="0 0 0"/>
-    <geometry>
-      <mesh filename="package://vica_description/meshes/lidar_1.stl" scale="0.001 0.001 0.001"/>
-    </geometry>
-  </collision>
+  <!-- No collision: a lidar has nothing to collide with, and the STL becomes a
+       convex hull on Isaac import that the scan then sees as an obstacle. -->
 </link>
 <link name="camera_link">

Commit message: fix(urdf): port canonical geometry from the real robot
Isaac was simulating a robot ~20% narrower than the real one. The drive wheel
joints sat at y = +/-0.1465 (0.293 m apart) against a tape-measured 0.364 m,
and the caster wheels were 10 mm inboard of their CAD position.

Values come from vica_ros2_ws@dev commit 621e181 and are expressed the same way
there: as formulas rather than constants. Every defect found in this model came
from a hand-copied number drifting away from its source, so the mesh origins now
derive from the frame they belong to.

  wheel_separation      0.364      (0.293)
  body_center_z         0.041      (0.0675)
  laser_z               0.192      (0.19)
  caster wheel dy       -0.005     (-0.015)
  base_link inertial z  0.03506... (0.00856...)

Collision offsets that used to compensate for the wrong joint positions are now
zero, which is the cross-check: with the joints correct, no compensation is
needed. The caster steer brackets lose their STL colliders for a box taken from
the CAD bounds, so nothing imports as a convex hull any more.

Caster colliders use 0.042 rather than the true 0.0375 radius. CAD leaves the
caster 4.5 mm off the ground; at the true radius PhysX rests the robot on its
drive wheels and pitches it ~0.635 deg back, tilting the lidar plane with it.

Expansion verified against the canonical model: wheel separation 0.364, caster
wheel at z 0.042, laser at 0.382, camera at 0.320, 11 links.

Still outstanding: add_drive_odom_graphs.py carries WHEEL_DISTANCE 0.293 and is
superseded by build_vica_ros_graphs.py, and the USD needs re-importing before
any of this reaches the simulator.

Co-Authored-By: Claude Opus 5 (1M context) <noreply@anthropic.com>

File: src/vica_description/urdf/VICA.xacro (robot description, xacro)
@@ -3,19 +3,32 @@
 <!-- Keep includes relative so this file expands before the package is installed. -->
 <xacro:include filename="materials.xacro" />
-<!-- Geometry exported from CAD is expressed in metres through a 0.001 mesh scale. -->
-<xacro:property name="body_center_z" value="0.0675" />
+<!-- Geometry exported from CAD is expressed in metres through a 0.001 mesh scale.
+     Coordinates below match vica_ros2_ws@dev (commit 621e181), which is the
+     canonical source: tape-measured on the robot and cross-checked against the
+     STL bounding boxes. Keep them as expressions, not constants; every bug
+     found in this model came from a hand-copied number drifting out of step. -->
+<xacro:property name="body_center_z" value="0.041" />
 <xacro:property name="base_link_height" value="0.19" />
 <!-- Simplified chassis collisions derived from the lower body and mast bounds. -->
 <xacro:property name="chassis_body_size" value="0.61 0.28 0.401" />
-<xacro:property name="chassis_body_origin" value="0 0 0.032" />
+<xacro:property name="chassis_body_origin" value="0 0 0.0585" />
 <xacro:property name="chassis_mast_size" value="0.24 0.04 0.414" />
-<xacro:property name="chassis_mast_origin" value="-0.385 0 0.4395" />
+<xacro:property name="chassis_mast_origin" value="-0.385 0 0.466" />
 <!-- Sensor origins are relative to base_link. -->
 <xacro:property name="laser_x" value="0.185" />
 <xacro:property name="laser_y" value="0.0" />
-<xacro:property name="laser_z" value="0.19" />
+<xacro:property name="laser_z" value="0.192" />
 <xacro:property name="camera_x" value="0.28683" />
 <xacro:property name="camera_y" value="0.0" />
-<xacro:property name="camera_z" value="0.13" />
+<xacro:property name="camera_z" value="0.130" />
+<!-- Wheel placement. wheel_separation is the measured centre-to-centre distance.
+     It is NOT the odometry constant. The real robot's encoder_feedback uses
+     wheel_base_m = 0.37, an effective tread fitted by rotation test that absorbs
+     tyre scrub. The two are different quantities and must not be unified. -->
+<xacro:property name="wheel_separation" value="0.364" />
+<xacro:property name="wheel_y" value="${wheel_separation / 2}" />
+<xacro:property name="caster_steer_y" value="0.0845" />
+<xacro:property name="caster_y" value="0.0795" />
+<xacro:property name="caster_wheel_dy" value="${round(caster_y - caster_steer_y, 6)}" />
 <!-- Conservative import defaults; tune these against the physical platform. -->
 <xacro:property name="wheel_effort" value="100.0" />
@@ -28,4 +41,9 @@
 <xacro:property name="caster_wheel_radius" value="0.0375" />
 <xacro:property name="caster_wheel_width" value="0.04" />
+<!-- CAD places the caster 4.5 mm clear of the ground, so a collider at the true
+     radius leaves PhysX resting the robot on its drive wheels and pitching it
+     ~0.635 deg back, tilting the lidar plane with it. Oversizing the collider by
+     that gap stands the robot level; the 4.5 mm stands in for tyre compression. -->
+<xacro:property name="caster_collision_radius" value="0.042" />
 <link name="base_footprint"/>
 <joint name="base_footprint_joint" type="fixed">
@@ -36,5 +54,5 @@
 <link name="base_link">
   <inertial>
-    <origin xyz="0.004031215194176557 3.002726997808124e-17 0.00856562657816282" rpy="0 0 0"/>
+    <origin xyz="0.004031215194176557 3.002726997808124e-17 0.03506562657816282" rpy="0 0 0"/>
     <mass value="90.84709962539795"/>
     <inertia ixx="2.402108" iyy="3.622523" izz="4.166828" ixy="0.0" iyz="-0.0" ixz="0.343284"/>
@@ -68,5 +86,5 @@
   </inertial>
   <visual>
-    <origin xyz="-0.154 -0.1465 0.084" rpy="0 0 0"/>
+    <origin xyz="-0.154 ${-wheel_y} 0.084" rpy="0 0 0"/>
     <geometry>
       <mesh filename="package://vica_description/meshes/left_wheel_1.stl" scale="0.001 0.001 0.001"/>
@@ -76,5 +94,5 @@
   <collision>
     <!-- URDF cylinders are Z-aligned; rotate onto this wheel's Y axis. -->
-    <origin xyz="0 0.0349 0" rpy="${pi / 2} 0 0"/>
+    <origin xyz="0 0 0" rpy="${pi / 2} 0 0"/>
     <geometry>
       <cylinder radius="${drive_wheel_radius}" length="${drive_wheel_width}"/>
@@ -89,5 +107,5 @@
   </inertial>
   <visual>
-    <origin xyz="-0.154 0.1465 0.084" rpy="0 0 0"/>
+    <origin xyz="-0.154 ${wheel_y} 0.084" rpy="0 0 0"/>
     <geometry>
       <mesh filename="package://vica_description/meshes/right_wheel_1.stl" scale="0.001 0.001 0.001"/>
@@ -97,5 +115,5 @@
   <collision>
     <!-- URDF cylinders are Z-aligned; rotate onto this wheel's Y axis. -->
-    <origin xyz="0 -0.0339 0" rpy="${pi / 2} 0 0"/>
+    <origin xyz="0 0 0" rpy="${pi / 2} 0 0"/>
     <geometry>
       <cylinder radius="${drive_wheel_radius}" length="${drive_wheel_width}"/>
@@ -110,5 +128,5 @@
   </inertial>
   <visual>
-    <origin xyz="0.252 -0.0695 0.107" rpy="0 0 0"/>
+    <origin xyz="0.252 ${-caster_y} 0.107" rpy="0 0 0"/>
     <geometry>
       <mesh filename="package://vica_description/meshes/front_left_caster_wheel_1.stl" scale="0.001 0.001 0.001"/>
@@ -118,7 +136,7 @@
   <collision>
     <!-- URDF cylinders are Z-aligned; rotate onto this wheel's Y axis. -->
-    <origin xyz="0 0.01 0" rpy="${pi / 2} 0 0"/>
-    <geometry>
-      <cylinder radius="${caster_wheel_radius}" length="${caster_wheel_width}"/>
+    <origin xyz="0 0 0" rpy="${pi / 2} 0 0"/>
+    <geometry>
+      <cylinder radius="${caster_collision_radius}" length="${caster_wheel_width}"/>
     </geometry>
   </collision>
@@ -131,5 +149,5 @@
   </inertial>
   <visual>
-    <origin xyz="0.252 0.0695 0.107" rpy="0 0 0"/>
+    <origin xyz="0.252 ${caster_y} 0.107" rpy="0 0 0"/>
     <geometry>
       <mesh filename="package://vica_description/meshes/front_right_caster_wheel_1.stl" scale="0.001 0.001 0.001"/>
@@ -139,7 +157,7 @@
   <collision>
     <!-- URDF cylinders are Z-aligned; rotate onto this wheel's Y axis. -->
-    <origin xyz="0 -0.01 0" rpy="${pi / 2} 0 0"/>
-    <geometry>
-      <cylinder radius="${caster_wheel_radius}" length="${caster_wheel_width}"/>
+    <origin xyz="0 0 0" rpy="${pi / 2} 0 0"/>
+    <geometry>
+      <cylinder radius="${caster_collision_radius}" length="${caster_wheel_width}"/>
     </geometry>
   </collision>
@@ -152,5 +170,5 @@
   </inertial>
   <visual>
-    <origin xyz="0.222 0.0845 0.0415" rpy="0 0 0"/>
+    <origin xyz="0.222 ${caster_steer_y} 0.0415" rpy="0 0 0"/>
     <geometry>
       <mesh filename="package://vica_description/meshes/front_right_caster_steer_1.stl" scale="0.001 0.001 0.001"/>
@@ -159,7 +177,8 @@
   </visual>
   <collision>
-    <origin xyz="0.222 0.0845 0.0415" rpy="0 0 0"/>
-    <geometry>
-      <mesh filename="package://vica_description/meshes/front_right_caster_steer_1.stl" scale="0.001 0.001 0.001"/>
+    <!-- CAD bounding box of the steer bracket; the STL became a convex hull on import. -->
+    <origin xyz="0 0 0.003" rpy="0 0 0"/>
+    <geometry>
+      <box size="0.08 0.08 0.0755"/>
     </geometry>
   </collision>
@@ -172,5 +191,5 @@
   </inertial>
   <visual>
-    <origin xyz="0.222 -0.0845 0.0415" rpy="0 0 0"/>
+    <origin xyz="0.222 ${-caster_steer_y} 0.0415" rpy="0 0 0"/>
     <geometry>
       <mesh filename="package://vica_description/meshes/front_left_caster_steer_1.stl" scale="0.001 0.001 0.001"/>
@@ -179,7 +198,8 @@
   </visual>
   <collision>
-    <origin xyz="0.222 -0.0845 0.0415" rpy="0 0 0"/>
-    <geometry>
-      <mesh filename="package://vica_description/meshes/front_left_caster_steer_1.stl" scale="0.001 0.001 0.001"/>
+    <!-- CAD bounding box of the steer bracket; the STL became a convex hull on import. -->
+    <origin xyz="0 0 0.003" rpy="0 0 0"/>
+    <geometry>
+      <box size="0.08 0.08 0.0755"/>
     </geometry>
   </collision>
@@ -192,5 +212,5 @@
   </inertial>
   <visual>
-    <origin xyz="-0.185 -0.0 -0.258" rpy="0 0 0"/>
+    <origin xyz="-0.185 -0.0 ${-(laser_z + body_center_z)}" rpy="0 0 0"/>
     <geometry>
       <mesh filename="package://vica_description/meshes/lidar_1.stl" scale="0.001 0.001 0.001"/>
@@ -214,5 +234,5 @@
 <link name="camera_optical_frame"/>
 <joint name="left_wheel_joint" type="continuous">
-  <origin xyz="0.154 0.1465 -0.125" rpy="0 0 0"/>
+  <origin xyz="0.154 ${wheel_y} -0.125" rpy="0 0 0"/>
   <parent link="base_link"/>
   <child link="left_wheel_1"/>
@@ -222,5 +242,5 @@
 </joint>
 <joint name="right_wheel_joint" type="continuous">
-  <origin xyz="0.154 -0.1465 -0.125" rpy="0 0 0"/>
+  <origin xyz="0.154 ${-wheel_y} -0.125" rpy="0 0 0"/>
   <parent link="base_link"/>
   <child link="right_wheel_1"/>
@@ -230,5 +250,5 @@
 </joint>
 <joint name="front_left_caster_wheel_joint" type="continuous">
-  <origin xyz="-0.03 -0.015 -0.0655" rpy="0 0 0"/>
+  <origin xyz="-0.03 ${caster_wheel_dy} -0.0655" rpy="0 0 0"/>
   <parent link="front_left_caster_steer_1"/>
   <child link="front_left_caster_wheel_1"/>
@@ -236,5 +256,5 @@
 </joint>
 <joint name="front_right_caster_wheel_joint" type="continuous">
-  <origin xyz="-0.03 0.015 -0.0655" rpy="0 0 0"/>
+  <origin xyz="-0.03 ${-caster_wheel_dy} -0.0655" rpy="0 0 0"/>
   <parent link="front_right_caster_steer_1"/>
   <child link="front_right_caster_wheel_1"/>
@@ -242,5 +262,5 @@
 </joint>
 <joint name="front_right_caster_steer_joint" type="continuous">
-  <origin xyz="-0.222 -0.0845 -0.087" rpy="0 0 0"/>
+  <origin xyz="-0.222 ${-caster_steer_y} -0.0825" rpy="0 0 0"/>
   <parent link="base_link"/>
   <child link="front_right_caster_steer_1"/>
@@ -248,5 +268,5 @@
 </joint>
 <joint name="front_left_caster_steer_joint" type="continuous">
-  <origin xyz="-0.222 0.0845 -0.087" rpy="0 0 0"/>
+  <origin xyz="-0.222 ${caster_steer_y} -0.0825" rpy="0 0 0"/>
   <parent link="base_link"/>
   <child link="front_left_caster_steer_1"/>

Commit message: feat(isaac): publish the camera under its RealSense names
The graphs published /rgb, /depth and /camera_info -- names that describe
what the topics are, and that nothing on the robot subscribes to. Use the
names realsense2_camera produces instead:

    /camera/camera/color/image_raw
    /camera/camera/color/camera_info
    /camera/camera/depth/image_rect_raw
    /camera/camera/depth/camera_info

vica_nvblox_bringup remaps all four by name, so this is the difference
between running nvblox against the simulator unmodified and maintaining a
second launch file whose behaviour is then not evidence about the robot.

Two camera_info publishers rather than one. Colour and depth are different
imagers with different intrinsics; the driver publishes both, and a consumer
that rectifies depth against colour intrinsics gets a subtly wrong cloud.

Frame ids follow the same rule, which reverses a comment this file used to
carry. It said not to use camera_color_optical_frame because the RealSense
driver owns that name and the publishers would collide. That is true on the
robot and backwards here: Isaac runs no driver, so unless VICA.xacro
declares those frames nothing can resolve the image headers at all. Add
camera_color_optical_frame and camera_depth_optical_frame there, with a note
that they are simulation-only for exactly that reason.

Both sit at camera_link, ignoring the baseline between the D455's colour and
depth imagers that the real driver reports. Harmless for costmaps at this
range; verify before trusting close-up colour-to-depth registration.

Verified: 28 graph nodes build against the hospital stage, and TF resolves
both new frames at [0.287, 0.000, 0.320], the measured camera height.

Co-Authored-By: Claude Opus 5 (1M context) <noreply@anthropic.com>

File: src/vica_description/urdf/VICA.xacro (robot description, xacro)
@@ -233,4 +233,16 @@
 </link>
 <link name="camera_optical_frame"/>
+<!-- The RealSense driver publishes camera_color_optical_frame and
+     camera_depth_optical_frame at runtime, so the physical robot's URDF must
+     not declare them: two publishers for one frame is a TF fight.
+     Isaac runs no driver, so here the URDF is the only thing that can supply
+     them, and it has to: the image headers coming out of the Isaac graphs
+     carry those frame names, and nvblox subscribes by them.
+     Simplification: both sit at camera_link, ignoring the few-centimetre
+     baseline between the D455's colour and depth imagers that the real driver
+     reports. Harmless for costmaps at this range; check it before trusting
+     close-up colour-to-depth registration. -->
+<link name="camera_color_optical_frame"/>
+<link name="camera_depth_optical_frame"/>
 <joint name="left_wheel_joint" type="continuous">
   <origin xyz="0.154 ${wheel_y} -0.125" rpy="0 0 0"/>
@@ -290,3 +302,15 @@
   <child link="camera_optical_frame"/>
 </joint>
+<!-- Same rotation, under the names the RealSense driver would publish. See the
+     note at the link declarations for why these exist only in simulation. -->
+<joint name="camera_color_optical_joint" type="fixed">
+  <origin xyz="0 0 0" rpy="-${pi / 2} 0 -${pi / 2}"/>
+  <parent link="camera_link"/>
+  <child link="camera_color_optical_frame"/>
+</joint>
+<joint name="camera_depth_optical_joint" type="fixed">
+  <origin xyz="0 0 0" rpy="-${pi / 2} 0 -${pi / 2}"/>
+  <parent link="camera_link"/>
+  <child link="camera_depth_optical_frame"/>
+</joint>
 </robot>

File: src/vica_description/urdf/vica.urdf (robot description, URDF)
Before this commit: robot VICA, 11 links, 10 joints
Links:
- added link camera_color_optical_frame
- added link camera_depth_optical_frame
Joints:
- added joint camera_color_optical_joint: type fixed, parent camera_link, child camera_color_optical_frame, origin xyz=0 0 0 rpy=-1.5707963267948966 0 -1.5707963267948966
- added joint camera_depth_optical_joint: type fixed, parent camera_link, child camera_depth_optical_frame, origin xyz=0 0 0 rpy=-1.5707963267948966 0 -1.5707963267948966
