Commit message: feat(urdf): put the camera on the handle post, and rebuild the stages
The sim robot still carried the camera at the old front mounting, 0.320 m
off the ground, long after vica_ros2_ws@dev moved it onto the handle post.
A depth camera 0.7 m from where the URDF says it is projects the floor into
the world at that offset, which is how a floor becomes a waist-high wall in
nvblox.

  camera_x  0.28683 -> -0.225   flush with the post's front face
  camera_z  0.130   ->  0.810   absolute 1.000 m (user's decision)

The mast collider went with it. Its old bounds described base_link.stl,
whose post stopped at 0.863 and ran back to -0.505; the redesigned body
reaches 1.075 and starts at -0.478. Read off the STL, not a drawing. The
visual mesh is base_link_mast.stl, copied from vica_ros2_ws@dev (55e1b0f).

Rebuilt through the whole chain rather than by hand: export_isaac_urdf.sh,
import_urdf_to_usd.py, then make_stage.sh for the hospital, corner and
avoid courses. All three pass verify_stage -- 13 checks each, including the
8-second play that catches a robot falling through the floor.

** The real robot has since been tape-measured three times and none of them
is 1.000 m: it now reads 1.045 with a 0.7 degree upward pitch that this
repository does not model. The gap is recorded in VICA.xacro's comment.
Anything measured on these stages was measured against a 1.000 m camera.

Co-Authored-By: Claude Opus 5 (1M context) <noreply@anthropic.com>
Claude-Session: https://claude.ai/code/session_01UMvK366QiL7tEMqZyyF3HS

File: src/vica_description/urdf/VICA.xacro (robot description, xacro)
@@ -86,13 +86,43 @@
      is ever regenerated from CAD. -->
 <xacro:property name="chassis_deck_measured_z" value="0.170" />
-<xacro:property name="chassis_mast_size" value="0.24 0.04 0.414" />
-<xacro:property name="chassis_mast_origin" value="-0.385 0 0.466" />
+<!-- The handle post, as the redesign leaves it. Bounds read off
+     meshes/base_link_mast.stl rather than copied from a drawing:
+       x  -0.478 .. -0.238   (0.24 deep, centre -0.358)
+       z   0.259 ..  0.885   base_link relative, absolute 0.449 .. 1.075
+     The old numbers described base_link.stl, whose post stopped at 0.863
+     absolute and ran back to -0.505. A collider still standing there would
+     have put a wall behind the robot that the render does not show. -->
+<xacro:property name="chassis_mast_size" value="0.24 0.04 0.626" />
+<xacro:property name="chassis_mast_origin" value="-0.358 0 0.572" />
 <!-- Sensor origins are relative to base_link. -->
 <xacro:property name="laser_x" value="0.185" />
 <xacro:property name="laser_y" value="0.0" />
 <xacro:property name="laser_z" value="0.192" />
-<xacro:property name="camera_x" value="0.28683" />
+<!-- Camera moved onto the handle post, following vica_ros2_ws@dev 6cb71a9.
+       camera_x  0.28683 -> -0.225   back 512 mm
+       camera_z  0.130   ->  0.810   absolute 1.000 m
+     x puts the 26 mm deep camera box's back face on -0.238, which is the
+     post's front face above. The two are flush, not guessed.
+     The height is 1.000 m by decision, taken when nothing had been measured
+     and vica_ros2_ws@dev still carried the 2026-08-18 design value 0.885
+     (absolute 1.075).
+     [미검증] The real robot has been measured since, three times, and this
+     is not any of them. vica_ros2_ws@dev now reads:
+         2026-08-24   ground 0.910   camera_z 0.720   first tape measure
+         2026-08-29   ground 1.025   camera_z 0.835
+         2026-08-30   ground 1.045   camera_z 0.855   after a remount
+     and it carries a camera_pitch of -0.0124 rad (0.7 degrees up, found by
+     fitting the floor plane in the depth cloud) that this file does not have
+     at all. So the sim robot sits 45 mm low and dead level while the real one
+     is 1.045 and tilted. That gap is a decision waiting to be made, not a
+     measurement waiting to be taken: matching it means rebuilding every stage
+     USD, and the courses in this repository were measured with the robot as
+     it stands here. Nothing downstream of this file has been re-run against
+     the real numbers. -->
+<!-- ** Anything measured on a stage built before that decision was measured
+     against a 1.000 m camera. Say so when the numbers are quoted. -->
+<xacro:property name="camera_x" value="-0.225" />
 <xacro:property name="camera_y" value="0.0" />
-<xacro:property name="camera_z" value="0.130" />
+<xacro:property name="camera_z" value="0.810" />
 <!-- Wheel placement. wheel_separation is the measured centre-to-centre distance.
      It is NOT the odometry constant. The real robot's encoder_feedback uses
@@ -163,8 +193,13 @@
     <inertia ixx="0.438065" iyy="0.660628" izz="0.759891" ixy="0.0" iyz="-0.0" ixz="0.062604"/>
   </inertial>
+  <!-- base_link_mast.stl, not base_link.stl: the same body with the rear
+       full-width rail and skirt cut away and the handle post carried up to
+       1.075 absolute, which is where the camera now mounts. Copied from
+       vica_ros2_ws@dev (55e1b0f). The collision below is still derived from
+       the primitives above, not from this mesh. -->
   <visual>
     <origin xyz="0 0 -${body_center_z}" rpy="0 0 0"/>
     <geometry>
-      <mesh filename="package://vica_description/meshes/base_link.stl" scale="0.001 0.001 0.001"/>
+      <mesh filename="package://vica_description/meshes/base_link_mast.stl" scale="0.001 0.001 0.001"/>
     </geometry>
     <material name="body_blue"/>

File: src/vica_description/urdf/vica.urdf (robot description, URDF)
Before this commit: robot VICA, 13 links, 12 joints
Links:
- link base_link: geometry collision box size=0.24 0.04 0.626; collision box size=0.61 0.28 0.401
Joints:
- joint camera_joint: origin xyz=0.28683 0.0 0.13 rpy=0 0 0 -> xyz=-0.225 0.0 0.81 rpy=0 0 0

File: src/vica_description/urdf/vica_arm.urdf (robot description, URDF)
Before this commit: robot VICA, 23 links, 22 joints
Links:
- link base_link: geometry collision box size=0.24 0.04 0.626; collision box size=0.61 0.28 0.401
Joints:
- joint camera_joint: origin xyz=0.28683 0.0 0.13 rpy=0 0 0 -> xyz=-0.225 0.0 0.81 rpy=0 0 0

Commit message: feat(sim): match the robot to the measured hardware, and open the controller matrix
Everything here exists so that a controller comparison run in simulation is
run against the robot that exists, not the one this repository remembered.

Robot
  camera_z 0.810 -> 0.855 (ground 1.045), the 2026-08-30 tape measure, and
  camera_pitch -0.0124 which this file did not model at all. The tilt matters
  in sim for the reason it matters on the robot: the depth camera hangs off
  camera_link, so 0.7 degrees the TF does not know about lifts the floor
  2.4 cm at 2 m and the costmap reads it as an obstacle.

  Two DYP-A22 ultrasonic probes on the front bumper, fitted 2026-08-31.
  Frames, and 20 mm cylinders so the mount is visible in a render. Visual
  only, ending flush with x = 0.305: that is the bumper face and the front of
  the footprint, and dev's comment is explicit that a probe past it means
  usonic_x and the footprint must both grow. [미검증] Nothing publishes into
  these frames in sim yet.

Footprint
  Tail -0.595 -> -0.415, half-width 0.2275 -> 0.225, following the robot's
  2026-08-29 measure (handle 19 -> 11 cm, body 80 -> 72 cm). The padded
  circumscribed radius drops 0.6506 -> 0.4727, so turn-in-place goes 1.30 ->
  0.95 m and inflation_radius 0.55 finally clears it. nav2 had been logging
  that shortfall every planner cycle and falling back to a full polygon check
  on every scored pose.

  That drop is also what makes MPPI admissible here at all. The robot's
  backlog put "inflation >= circumscribed" as a precondition on any
  controller that does not check the footprint itself.

Speeds
  max_vel_x 0.26 -> 0.5, max_vel_theta 0.4 -> 0.5, decel_lim_x -2.5 -> -1.5,
  sim_time 2.5 -> 2.0. All dev's. The old numbers were dev's too, three
  months ago; the note on the robot says 0.26 "너무 느렸다".

Controllers and planners
  Three controllers and four planners, selectable in one command. RPP is the
  robot's run1215 configuration, the one that arrived. Each block is named
  for what it is and select_controller renames the chosen pair to
  FollowPath/GridBased, which is what the behaviour tree asks for. Round
  trips are byte-identical.

A fourth course
  vica_uturncourse: dead-end corridors at 1.00/1.20/1.50/1.80/2.00, drive in,
  turn 180, drive out. Nothing else here asks the robot to reverse heading,
  and reversing heading is the requirement the robot failed on 2026-08-29.
  Corner and avoid courses move to 0.80/0.90/1.00/1.20/1.50.

Two repairs
  The hospital stage referenced its environment by a relative path, and the
  workspace moving from ~/vica_ws into VICA-smarthandle/ put that path one
  directory out. Colliders fell 134 -> 8, the floor among them, and the robot
  dropped 66.8 m. A full rebuild recomputes the path.

  make_stage.sh called that stage verified anyway. verify_stage.py reports
  the failure and calls sys.exit(1), but Isaac's SimulationApp.close() runs
  first and ends the process with status 0, so the exit code said pass and
  stamp_verified marked it. The harness accepts a stamped stage, so the next
  run would have produced a full table of numbers about a robot in freefall.
  The verify step now reads the log as well as the code -- the same guard the
  prepare step already had, and for the same reason.

** Every result recorded in this repository before today was measured with a
1.000 m camera, no tilt, and the longer body. None of it is comparable.

Co-Authored-By: Claude Opus 5 (1M context) <noreply@anthropic.com>
Claude-Session: https://claude.ai/code/session_01RnJpDRgBtMFe8arQPicSZr

File: src/vica_description/urdf/VICA.xacro (robot description, xacro)
@@ -99,30 +99,51 @@
 <xacro:property name="laser_y" value="0.0" />
 <xacro:property name="laser_z" value="0.192" />
-<!-- Camera moved onto the handle post, following vica_ros2_ws@dev 6cb71a9.
-       camera_x  0.28683 -> -0.225   back 512 mm
-       camera_z  0.130   ->  0.810   absolute 1.000 m
-     x puts the 26 mm deep camera box's back face on -0.238, which is the
-     post's front face above. The two are flush, not guessed.
-     The height is 1.000 m by decision, taken when nothing had been measured
-     and vica_ros2_ws@dev still carried the 2026-08-18 design value 0.885
-     (absolute 1.075).
-     [미검증] The real robot has been measured since, three times, and this
-     is not any of them. vica_ros2_ws@dev now reads:
+<!-- Camera on the handle post. Tracks vica_ros2_ws@dev, which is the source
+     of truth for robot geometry. This file follows it, never the reverse.
+       camera_x  -0.225   the 26 mm camera box's back face lands on -0.238,
+                          the post's front face above. Flush, not guessed.
+       camera_z   0.855   absolute 1.045 m
+     2026-09-02: matched to the real robot, replacing the 1.000 m that was
+     chosen here on 2026-08-24 when nothing had been tape-measured yet. The
+     robot has been measured three times since and the last one stands:
          2026-08-24   ground 0.910   camera_z 0.720   first tape measure
          2026-08-29   ground 1.025   camera_z 0.835
          2026-08-30   ground 1.045   camera_z 0.855   after a remount
-     and it carries a camera_pitch of -0.0124 rad (0.7 degrees up, found by
-     fitting the floor plane in the depth cloud) that this file does not have
-     at all. So the sim robot sits 45 mm low and dead level while the real one
-     is 1.045 and tilted. That gap is a decision waiting to be made, not a
-     measurement waiting to be taken: matching it means rebuilding every stage
-     USD, and the courses in this repository were measured with the robot as
-     it stands here. Nothing downstream of this file has been re-run against
-     the real numbers. -->
-<!-- ** Anything measured on a stage built before that decision was measured
-     against a 1.000 m camera. Say so when the numbers are quoted. -->
+     Re-measure on the robot before trusting this; it moves whenever the
+     camera is detached. The real config's comment carries the full history.
+     ** Every stage USD and every result recorded before 2026-09-02 was made
+     with the camera at 1.000 m and dead level. They are not comparable to
+     anything measured after. -->
 <xacro:property name="camera_x" value="-0.225" />
 <xacro:property name="camera_y" value="0.0" />
-<xacro:property name="camera_z" value="0.810" />
+<xacro:property name="camera_z" value="0.855" />
+<!-- The mast sits 0.7 degrees nose-up, measured on the real robot by fitting
+     the floor plane in the depth cloud (RANSAC, 3 runs, -2.35/-2.31/-2.24
+     degrees residual against a URDF that then said -3.0). Sign convention:
+     URDF pitch is positive down, so nose-up is negative.
+     It matters here for the same reason it matters on the robot. Isaac's
+     depth camera hangs off camera_link, so a tilt the TF does not know about
+     puts every returned point at the wrong height: at 2 m, 0.7 degrees is
+     2.4 cm, and the floor lifts into the costmap's slice as an obstacle.
+     Modelling the tilt costs nothing and removes a whole class of "the
+     corridor filled in" confusion from the comparison runs. -->
+<xacro:property name="camera_pitch" value="-0.0124" />
+<!-- Two DYP-A22 ultrasonic rangers on the front bumper, fitted to the robot
+     2026-08-31. Mounted horizontally; the housing cannot be tilted.
+     vica_ros2_ws@dev and docs/handoff_jetson_ultrasonic_i2c.md are the source.
+       x  0.305    the bumper face itself
+       y  +-0.107  either side of centre
+       z -0.0987   ground 0.0913, minus base_link_height 0.190
+     Frame names have to match the driver's ultrasonic_frame_ids, so they are
+     copied rather than invented.
+     Why they exist: the depth camera at 1.045 m looks over anything low and
+     close. These sit at ankle height where the lidar plane (0.382) and the
+     camera both have nothing to say. [미검증] in sim. The frames are here so
+     a range sensor can be attached to them, but no Isaac sensor is publishing
+     into them yet and no costmap layer consumes them. The comparison runs
+     below do not use ultrasound. -->
+<xacro:property name="usonic_x" value="0.305" />
+<xacro:property name="usonic_y" value="0.107" />
+<xacro:property name="usonic_z" value="-0.0987" />
 <!-- Wheel placement. wheel_separation is the measured centre-to-centre distance.
      It is NOT the odometry constant. The real robot's encoder_feedback uses
@@ -431,6 +452,41 @@
   <child link="laser_frame"/>
 </joint>
+<!-- The probe bodies, drawn so the mounting point is visible in a render
+     instead of being an invisible frame nobody can check.
+     DYP-A22 is a sealed cylindrical probe, 20 mm across and about 15 mm of
+     barrel proud of its mount. Modelled as a cylinder on the x axis, which is
+     the direction it looks; a URDF cylinder stands on z, so it is laid down
+     by a 90 degree pitch.
+     Placed to end flush with x = 0.305, not to stick out past it. That is the
+     bumper face and the front edge of the footprint, and vica_ros2_ws@dev's
+     comment is explicit that a probe protruding beyond it means usonic_x AND
+     the footprint front must both grow. Neither has grown on the robot, so
+     flush is what the robot's own numbers describe. If a tape measure says
+     otherwise, this mesh is the thing that was wrong, not the footprint.
+     Visual only. A 20 mm bump on the bumper face changes nothing the planner
+     reasons about, and giving it a collider would put a second obstacle
+     inside the footprint the robot already plans against. -->
+<xacro:property name="usonic_radius" value="0.010" />
+<xacro:property name="usonic_len" value="0.015" />
+<xacro:macro name="usonic_probe" params="name y">
+  <link name="${name}">
+    <visual>
+      <origin xyz="${-usonic_len/2} 0 0" rpy="0 ${pi/2} 0"/>
+      <geometry>
+        <cylinder radius="${usonic_radius}" length="${usonic_len}"/>
+      </geometry>
+      <material name="camera_black"/>
+    </visual>
+  </link>
+  <joint name="${name}_joint" type="fixed">
+    <origin xyz="${usonic_x} ${y} ${usonic_z}" rpy="0 0 0"/>
+    <parent link="base_link"/>
+    <child link="${name}"/>
+  </joint>
+</xacro:macro>
+<xacro:usonic_probe name="usonic_front_left"  y="${usonic_y}" />
+<xacro:usonic_probe name="usonic_front_right" y="${-usonic_y}" />
 <joint name="camera_joint" type="fixed">
-  <origin xyz="${camera_x} ${camera_y} ${camera_z}" rpy="0 0 0"/>
+  <origin xyz="${camera_x} ${camera_y} ${camera_z}" rpy="0 ${camera_pitch} 0"/>
   <parent link="base_link"/>
   <child link="camera_link"/>

File: src/vica_description/urdf/vica.urdf (robot description, URDF)
Before this commit: robot VICA, 13 links, 12 joints
Links:
- added link usonic_front_left; visual cylinder length=0.015 radius=0.01
- added link usonic_front_right; visual cylinder length=0.015 radius=0.01
Joints:
- added joint usonic_front_left_joint: type fixed, parent base_link, child usonic_front_left, origin xyz=0.305 0.107 -0.0987 rpy=0 0 0
- added joint usonic_front_right_joint: type fixed, parent base_link, child usonic_front_right, origin xyz=0.305 -0.107 -0.0987 rpy=0 0 0
- joint camera_joint: origin xyz=-0.225 0.0 0.81 rpy=0 0 0 -> xyz=-0.225 0.0 0.855 rpy=0 -0.0124 0

File: src/vica_description/urdf/vica_arm.urdf (robot description, URDF)
Before this commit: robot VICA, 23 links, 22 joints
Links:
- added link usonic_front_left; visual cylinder length=0.015 radius=0.01
- added link usonic_front_right; visual cylinder length=0.015 radius=0.01
Joints:
- added joint usonic_front_left_joint: type fixed, parent base_link, child usonic_front_left, origin xyz=0.305 0.107 -0.0987 rpy=0 0 0
- added joint usonic_front_right_joint: type fixed, parent base_link, child usonic_front_right, origin xyz=0.305 -0.107 -0.0987 rpy=0 0 0
- joint camera_joint: origin xyz=-0.225 0.0 0.81 rpy=0 0 0 -> xyz=-0.225 0.0 0.855 rpy=0 -0.0124 0

Commit message: fix(urdf): give the ultrasonic probes mass, and make verify catch it next time
The probes were added with visual geometry and no <inertial>. The URDF
importer runs with merge_fixed_joints off, so a link carrying geometry becomes
its own rigid body rather than folding into base_link, and a rigid body with
no inertial gets no mass at all. Body count went 9 to 11 and two of the new
ones were massless.

That took the articulation's mass matrix with it. The symptom was not a crash:

    wheel joints    -1.16 / 2.35 rad, turning steadily
    /cmd_vel        0.26 m/s, arriving at 20 Hz
    /odom x         2.4e-07 m
    /odom z         -0.021 m, sunk into the floor

Wheels turning, body still. camera_link has been massless all along and the
robot drove fine; one it tolerated, three it did not.

30 g each, which is the probe and its lead.

The reason this ran for an hour before anyone noticed is the more useful half.
verify_stage asked whether the robot stays put -- height steady, no drift, no
NaN -- and a robot that cannot move passes every one of those with full marks.
It was stamped verified and handed to the screening run, which scored zero on
every cell it reached.

So verify_stage now also commands the wheels directly and requires the body to
translate: 4 rad/s for 3 seconds, at least 0.10 m. No ROS, no controller, no
map. The corner stage does 0.521 m, against the 0.26 m/s the wheel radius
predicts. If this check fails nothing downstream is worth running, and it
fails in ninety seconds instead of three hours.

Co-Authored-By: Claude Opus 5 (1M context) <noreply@anthropic.com>
Claude-Session: https://claude.ai/code/session_01RnJpDRgBtMFe8arQPicSZr

File: src/vica_description/urdf/VICA.xacro (robot description, xacro)
@@ -471,4 +471,17 @@
 <xacro:macro name="usonic_probe" params="name y">
   <link name="${name}">
+    <!-- 30 g, the probe and its lead.
+         Not optional. The importer runs with merge_fixed_joints off, so a link
+         carrying geometry becomes its own rigid body rather than folding into
+         base_link, and a rigid body with no inertial gets no mass at all.
+         Two of those on fixed joints took the articulation's mass matrix with
+         them: the wheels turned, the body did not move, and it sank 21 mm into
+         the floor. Body count went 9 to 11 and the robot stopped driving.
+         camera_link gets away with it as the only one; two more did not. -->
+    <inertial>
+      <origin xyz="${-usonic_len/2} 0 0" rpy="0 0 0"/>
+      <mass value="0.03"/>
+      <inertia ixx="1.5e-6" iyy="1.5e-6" izz="1.5e-6" ixy="0" iyz="0" ixz="0"/>
+    </inertial>
     <visual>
       <origin xyz="${-usonic_len/2} 0 0" rpy="0 ${pi/2} 0"/>

File: src/vica_description/urdf/vica.urdf (robot description, URDF)
Before this commit: robot VICA, 15 links, 14 joints
Links:
- link usonic_front_left: mass None -> 0.03
- link usonic_front_right: mass None -> 0.03

File: src/vica_description/urdf/vica_arm.urdf (robot description, URDF)
Before this commit: robot VICA, 25 links, 24 joints
Links:
- link usonic_front_left: mass None -> 0.03
- link usonic_front_right: mass None -> 0.03
