Commit message: fix(sim): the robot sank because of two things, and neither was the robot
PhysX had been naming one of them on every play, in a log nobody read:

    The rigid body at .../base_link/camera_link has a possibly invalid
    inertia tensor of {1.0, 1.0, 1.0} and a negative mass

camera_link carried visual geometry, a fixed joint and no <inertial>. With
merge_fixed_joints off that is a rigid body with nothing to weigh. An
articulation solves as one system, so a negative mass in one link is not
confined to that link: the robot settled 6 mm low and 2.4 degrees nose-up in
places where it should have been level. This is the same defect the ultrasonic
probes had in 912d8ba, and a comment added there said camera_link could get
away with it. It could not.

The other was the floor. Each course floored itself with one 50 m box, and the
chassis box collided with it while the 65 mm wheel cylinders did not -- at some
places along it and not others. Settling height along the corner course, one
change between the rows:

    floor box     -22 0.183  -8.65 0.190  -4.3 0.171  0 0.142
                  +8.65 0.142  +13 0.142  +22 0.170
    ground plane  all seven 0.190

0.190 is the wheels carrying the robot; 0.142 is the chassis on the floor with
the wheels 48 mm underground. At x=0 they spun 5050 degrees in 14 s and the
robot moved 0.000 m. The floor box stays for the renders and the depth camera;
a purpose=guide plane does the colliding.

With both fixed, ten spawn positions all settle at 0.190 with zero roll and
pitch, and commanded 2, 4, 6 and 8 rad/s all come back as 100 per cent of
r*omega with no slip.

verify_stage now reads every rigid body's mass and requires the ground plane,
because none of its existing checks could see either fault: the body count was
right, the bodies had joints, and the play check only ever stands the robot on
one spot. set_mass_from_urdf can now create a MassAPI that is missing rather
than walking past the body that has none, which is why --check reported
"차이 없음" while the two totals differed by camera_link's 0.113 kg.

Two comments in fixup_vica_usd_joints are corrected rather than deleted. They
asserted sleep and then missing cylinder shapes as the cause; both are wrong,
and PhysX does carry cylinders as custom geometry. The settings stay, on their
own merits, with what was actually measured written down. set_stage_spawn.py
is deleted: it existed only to work around a cause that was not one.

Co-Authored-By: Claude Opus 5 (1M context) <noreply@anthropic.com>
Claude-Session: https://claude.ai/code/session_01RnJpDRgBtMFe8arQPicSZr

File: src/vica_description/urdf/VICA.xacro (robot description, xacro)
@@ -384,4 +384,21 @@
 <link name="camera_link">
   <!-- RViz placeholder; Isaac Sim uses its own D455 USD sensor asset. -->
+  <!-- 113 g, the D455's datasheet mass.
+       Not optional, for the same reason the ultrasonic links say so: with
+       merge_fixed_joints off, a link carrying geometry becomes its own rigid
+       body, and a rigid body with no inertial gets no mass. PhysX then reports
+       "possibly invalid inertia tensor of {1.0, 1.0, 1.0} and a negative mass"
+       on every play, and the articulation's mass matrix goes with it. The
+       symptom is position dependent and looks like anything but a mass bug:
+       at x=-22 the wheels would not turn and the body slid 0.38 m and stopped,
+       at x=0 the wheels spun 5050 degrees while the body never moved and sat
+       48 mm low with its chassis on the floor. An earlier comment here claimed
+       camera_link could get away with having no inertial. It could not. -->
+  <inertial>
+    <origin xyz="0 0 0" rpy="0 0 0"/>
+    <mass value="0.113"/>
+    <inertia ixx="1.53e-4" iyy="1.43e-5" izz="1.51e-4"
+             ixy="0.0" iyz="0.0" ixz="0.0"/>
+  </inertial>
   <visual>
     <origin xyz="0 0 0" rpy="0 0 0"/>
@@ -478,5 +495,5 @@
          them: the wheels turned, the body did not move, and it sank 21 mm into
          the floor. Body count went 9 to 11 and the robot stopped driving.
-         camera_link gets away with it as the only one; two more did not. -->
+         camera_link had the same defect and the same excuse; see its link. -->
     <inertial>
       <origin xyz="${-usonic_len/2} 0 0" rpy="0 0 0"/>

File: src/vica_description/urdf/vica.urdf (robot description, URDF)
Before this commit: robot VICA, 15 links, 14 joints
Links:
- link camera_link: mass None -> 0.113

Commit message: feat(urdf): OpenMANIPULATOR-X 를 관절까지 모델링하고, 늘릴 수 있게 한다
요청받은 팔이다. 기존 arm 변형은 Kinova Gen3 lite 를 질량 덩어리로만 들고
있었고 관절이 없었다. arm_model 로 갈라, 기본은 omx 이고 gen3_lite 는 남는다 —
라이저 높이를 정한 계산이 Gen3 기준이라 그 기록이 아직 유효하다.

기하·관절한계·링크질량은 ROBOTIS 의 open_manipulator_x_description (humble
브랜치) 에서 옮겼다. 포함(include)하지 않고 옮겨 적은 이유는 셋이다.

  - 그 패키지가 여기 설치돼 있지 않고, 설치는 승인 항목이다. VICA.xacro 는
    주행만 하는 모든 기계에서 확장돼야 하고 거기엔 로봇 본체도 포함된다.
  - 길이를 우리가 바꿔야 한다. 남의 패키지 안의 상수로는 못 바꾼다.
  - 메시가 이 워크스페이스에 없다. 그래서 그린 것은 관절 간격으로 크기를 맞춘
    상자와 원기둥이다. 운동학과 질량은 ROBOTIS 의 숫자, 모양은 근사다.

왜 늘려야 하는가는 계산했다. 확장된 URDF 에서 네 관절을 각자의 한계 안에서
훑어 도달점을 샘플링했고, 데크 0.449 m + 라이저 0.10 기준:

    l3 / l4        최고높이   1.10 m 전방   코 끝(x=+0.305) 기준
    0.128 / 0.124   0.915     닿지 않음         -
    0.20  / 0.20    1.061     닿지 않음         -
    0.25  / 0.25    1.161      +0.311        +6 mm
    0.30  / 0.28    1.241      +0.456       +151 mm

기본 OMX 는 엘리베이터 버튼 1.10 m 에 어떤 자세로도 못 닿는다. 0.25/0.25 는
닿지만 그리퍼가 로봇 코보다 6 mm 앞이라 벽에 붙어야 한다. 0.30/0.28 이
라이저를 올리지 않고 151 mm 를 벌어주는 첫 줄이고, 무게중심을 높이지 않는다.

그 값은 기본값이 아니라 플래그다. 파일은 ROBOTIS 가 파는 물건을 계속 기술해야
한다. export_isaac_urdf.sh 는 VICA_ARM_ARGS 로 받는다:

    VICA_ARM_ARGS="arm_link3_len:=0.30 arm_link4_len:=0.28" \
        export_isaac_urdf.sh --arm

include 는 $(find vica_description) 가 아니라 상대 경로다. find 형은
AMENT_PREFIX_PATH 에 워크스페이스가 있어야 하는데 export_isaac_urdf.sh 는 ROS 만
source 한 기계에서도 돌아야 하고, 실제로 그 자리에서 깨졌다.

Co-Authored-By: Claude Opus 5 (1M context) <noreply@anthropic.com>
Claude-Session: https://claude.ai/code/session_01RnJpDRgBtMFe8arQPicSZr

File: src/vica_description/urdf/VICA.xacro (robot description, xacro)
@@ -23,10 +23,8 @@
          export_isaac_urdf.sh          -> urdf/vica.urdf
          export_isaac_urdf.sh (arm)    -> urdf/vica_arm.urdf
-     The arm is a Kinova Gen3 lite on a riser. [미검증] What is
-     modelled here is its mass and its stowed envelope, not its
-     kinematics: the six joints need kortex_description, which is
-     not in this workspace and whose installation is an approval
-     item. So use_arm:=true today gives a robot that weighs and
-     balances like the real thing and cannot move an elbow.
+     arm_model:=omx is the default and is the direction the
+     project is going: an OpenMANIPULATOR~X with real joints and
+     lengths we can change. arm_model:=gen3_lite still gives the
+     Kinova the riser numbers below were chosen against.
      That split is deliberate rather than a shortcut. Everything the
      driving stack cares about is the stowed case: the footprint it
@@ -55,4 +53,43 @@
 <xacro:arg name="arm_riser_h" default="0.10" />
 <xacro:property name="arm_riser_h" value="$(arg arm_riser_h)" />
+<!-- Which arm. omx is the OpenMANIPULATOR-X the project is moving to;
+     gen3_lite is the Kinova the riser numbers above were worked out against,
+     kept because those numbers are still the record of how the riser was
+     chosen and because kortex_description is installed.
+     They are not interchangeable in reach. The Gen3 lite goes 0.76 m and the
+     OMX 0.38, so an OMX on a 0.449 m deck with a 0.10 m riser tops out near
+     0.93 m and a lift button at 1.10 is out of the question as bought. The
+     three lengths below exist for that: the plan is to lengthen the arm in
+     our own design, and this is where the design gets tried before it is
+     built. urdf/omx_arm.xacro says what scales with them. -->
+<xacro:arg name="arm_model" default="omx" />
+<xacro:property name="arm_model" value="$(arg arm_model)" />
+<!-- Stock OMX: 0.128 upper arm, 0.124 forearm, 0.126 wrist to tip.
+     Left at stock so that arm_model:=omx describes the arm as bought. What it
+     costs is measured rather than guessed: sampling the four joints over their
+     own limits from the expanded URDF, with the deck at 0.449 m and the riser
+     at 0.10, the tip tops out at 0.915 m. A lift button at 1.10 is not
+     reachable at all, in any pose.
+     What lengthening buys, same sampling, forward reach taken at 1.10 m and
+     the robot's own front edge at x = +0.305:
+         l3 / l4       riser   최고높이   1.10 m 전방   코 끝 기준
+         0.128 / 0.124  0.10    0.915     닿지 않음        -
+         0.20  / 0.20   0.10    1.061     닿지 않음        -
+         0.25  / 0.25   0.10    1.161      +0.311        +6 mm
+         0.30  / 0.28   0.10    1.241      +0.456       +151 mm
+         0.30  / 0.28   0.20    1.341      +0.548       +243 mm
+     0.25/0.25 reaches the button and the gripper is 6 mm past the robot's own
+     nose, so the robot would have to be touching the wall. 0.30/0.28 on the
+     same 0.10 riser stands 151 mm off it, which is the first row that is
+     actually usable, and it buys that without raising the centre of mass.
+     Raising the riser instead is the more expensive way to the same place:
+     mass at the top of the robot is what the forward tipping margin pays for,
+     and scripts/mass_properties.py prints that.
+     So the design number to try is arm_link3_len:=0.30 arm_link4_len:=0.28,
+     and it is a flag rather than an edit because it is not what ROBOTIS
+     sells. -->
+<xacro:arg name="arm_link3_len" default="0.128" />
+<xacro:arg name="arm_link4_len" default="0.124" />
+<xacro:arg name="arm_link5_len" default="0.126" />
 <!-- Geometry exported from CAD is expressed in metres through a 0.001 mesh scale.
      Coordinates below match vica_ros2_ws@dev (commit 621e181), which is the
@@ -660,17 +697,47 @@
        written for a real arm on a network. Nothing in simulation reads them.
        0.0.0.0 is there to be obviously not an address. -->
-  <xacro:include filename="$(find kortex_description)/arms/gen3_lite/6dof/urdf/gen3_lite_macro.xacro" />
-  <xacro:load_arm
-      parent="arm_mount_link"
-      prefix="gen3_"
-      dof="6"
-      vision="false"
-      robot_ip="0.0.0.0"
-      gripper_joint_name="gen3_gripper"
-      use_fake_hardware="true"
-      sim_isaac="false"
-      sim_gazebo="false">
-    <origin xyz="0 0 0" rpy="0 0 0"/>
-  </xacro:load_arm>
+  <xacro:if value="${arm_model == 'omx'}">
+    <!-- Transcribed rather than included, for the three reasons omx_arm.xacro
+         gives at length. The short one: the package is not installed here and
+         the lengths have to be ours to change. -->
+    <!-- Relative, not $(find vica_description). The find form needs the
+         workspace on AMENT_PREFIX_PATH, and export_isaac_urdf.sh is supposed
+         to run on a machine that has only sourced ROS, and it broke there the
+         moment this include was added. Relative resolves against this file. -->
+    <xacro:include filename="omx_arm.xacro" />
+    <xacro:omx_arm parent="arm_mount_link" prefix="omx_"
+                   link3_len="$(arg arm_link3_len)"
+                   link4_len="$(arg arm_link4_len)"
+                   link5_len="$(arg arm_link5_len)">
+      <origin xyz="0 0 0" rpy="0 0 0"/>
+    </xacro:omx_arm>
+  </xacro:if>
+  <xacro:if value="${arm_model == 'gen3_lite'}">
+    <!-- ros-jazzy-kortex-description 0.2.6.
+         The include lives inside these guards on purpose. VICA.xacro has to
+         expand on a machine that has never heard of kortex_description, which
+         is every machine that only drives, including the physical robot's. At
+         the top of the file the include would run unconditionally and
+         use_arm:=false would stop working there.
+         prefix is not decoration. The macro names its own root
+         "${prefix}base_link", and this robot already has a base_link; without
+         a prefix the two collide and the arm silently reparents the chassis.
+         robot_ip and the gripper name are required parameters of a macro
+         written for a real arm on a network. Nothing in simulation reads them.
+         0.0.0.0 is there to be obviously not an address. -->
+    <xacro:include filename="$(find kortex_description)/arms/gen3_lite/6dof/urdf/gen3_lite_macro.xacro" />
+    <xacro:load_arm
+        parent="arm_mount_link"
+        prefix="gen3_"
+        dof="6"
+        vision="false"
+        robot_ip="0.0.0.0"
+        gripper_joint_name="gen3_gripper"
+        use_fake_hardware="true"
+        sim_isaac="false"
+        sim_gazebo="false">
+      <origin xyz="0 0 0" rpy="0 0 0"/>
+    </xacro:load_arm>
+  </xacro:if>
 </xacro:if>
 </robot>

File: src/vica_description/urdf/vica_arm.urdf (robot description, URDF)
Before this commit: robot VICA, 25 links, 24 joints
Links:
- removed link gen3_arm_link
- removed link gen3_base_link
- removed link gen3_dummy_link
- removed link gen3_end_effector_link
- removed link gen3_forearm_link
- removed link gen3_lower_wrist_link
- removed link gen3_shoulder_link
- removed link gen3_upper_wrist_link
- added link omx_end_effector_link
- added link omx_gripper_left_link, mass 0.012; visual box size=0.04 0.008 0.02
- added link omx_gripper_right_link, mass 0.012; visual box size=0.04 0.008 0.02
- added link omx_link1, mass 0.079119962; visual box size=0.045 0.045 0.034
- added link omx_link2, mass 0.098406837; visual box size=0.045 0.045 0.0595
- added link omx_link3, mass 0.32463086718749995; visual box size=0.045 0.045 0.3
- added link omx_link4, mass 0.29974817419354843; visual box size=0.28 0.045 0.045
- added link omx_link5, mass 0.14327573; visual box size=0.126 0.045 0.045
- link camera_link: mass None -> 0.113
Joints:
- removed joint gen3_base_joint
- removed joint gen3_end_effector
- removed joint gen3_joint_1
- removed joint gen3_joint_2
- removed joint gen3_joint_3
- removed joint gen3_joint_4
- removed joint gen3_joint_5
- removed joint gen3_joint_6
- added joint omx_base_joint: type fixed, parent arm_mount_link, child omx_link1, origin xyz=0 0 0 rpy=0 0 0
- added joint omx_end_effector_joint: type fixed, parent omx_link5, child omx_end_effector_link, origin xyz=0.126 0.0 0.0 rpy=0 0 0
- added joint omx_gripper_left_joint: type prismatic, parent omx_link5, child omx_gripper_left_link, origin xyz=0.081648 0.021 0.0 rpy=0 0 0, axis 0 1 0, limit lower=-0.010 upper=0.019 effort=1.0 velocity=0.5
- added joint omx_gripper_right_joint: type prismatic, parent omx_link5, child omx_gripper_right_link, origin xyz=0.081648 -0.021 0 rpy=0 0 0, axis 0 -1 0, limit lower=-0.010 upper=0.019 effort=1.0 velocity=0.5, mimic joint=omx_gripper_left_joint multiplier=1.0 offset=0.0
- added joint omx_joint1: type revolute, parent omx_link1, child omx_link2, origin xyz=0.012 0.0 0.017 rpy=0 0 0, axis 0 0 1, limit lower=-3.141592653589793 upper=3.141592653589793 effort=1.5 velocity=4.82
- added joint omx_joint2: type revolute, parent omx_link2, child omx_link3, origin xyz=0.0 0.0 0.0595 rpy=0 0 0, axis 0 1 0, limit lower=-1.5 upper=1.5 effort=1.5 velocity=4.82
- added joint omx_joint3: type revolute, parent omx_link3, child omx_link4, origin xyz=0.024 0 0.3 rpy=0 0 0, axis 0 1 0, limit lower=-1.5 upper=1.4 effort=1.5 velocity=4.82
- added joint omx_joint4: type revolute, parent omx_link4, child omx_link5, origin xyz=0.28 0.0 0.0 rpy=0 0 0, axis 0 1 0, limit lower=-1.7 upper=1.97 effort=1.5 velocity=4.82
