Commit message: feat(urdf): 팔을 VICA 높이에 맞춰 늘리고, 늘린 부분을 그린다
기본값이 0.30 / 0.28 이 됐다. 로보티스가 파는 길이로는 손끝이 0.915 m 에서
멈추고 엘리베이터 버튼은 1.10 m 라 어떤 자세로도 닿지 않는다. 0.30 / 0.28 이면
1.241 m 까지 올라가고 로봇 코 끝보다 151 mm 앞에서 누른다. 카탈로그 숫자가
필요할 때는 arm_link3_len:=0.128 arm_link4_len:=0.124 로 되돌린다.

막고 있던 것은 계산이 아니라 그림이었다. 로보티스 메시는 그들이 파는 길이
그대로라, 관절만 멀리 보내면 껍데기는 제자리에 남아 팔의 앞쪽 절반이 떨어져
떠 있는 것처럼 렌더됐다. 그래서 지난번에 기본 길이로 되돌렸다. 실제로 만들
물건이 "같은 모터 + 우리 링크" 이니 그림도 그렇게 그린다: 케이싱은 제 크기로,
늘린 만큼은 30x30x2 알루미늄 각봉으로. stock=0 은 그 링크가 안 늘어난다는
뜻이고, 이 검사가 없어서 link1 과 link2 는 케이싱 전체에 봉이 덧그려졌다 —
아무것도 nothing 보다는 길기 때문이다.

질량을 길이에 정비례로 늘리던 것을 케이싱 + 0.60 kg/m 로 바꿨다. 로보티스
138 g 의 대부분은 양 끝 브래킷이고 브래킷은 길어지지 않는다. 예전 모델은 어깨
토크를 15% 과장했다.

늘어난 대가는 전복이 아니라 어깨 모터다. 전방 전복은 7.84 에서 6.44 m/s² 로,
제동 한계의 2.57 배라 여유가 있다. joint2 는 다르다: 수평으로 곧게 뻗으면 팔
자체가 2.80 N.m 로 XM430 스톨의 68% 이고, 500 g 을 얹으면 6.56 로 모터가 가진
것의 한 배 반이다. 긴 팔은 버튼을 누르고 짐은 못 든다. 그 숫자는 주석이 아니라
scripts/arm_torque.py 가 확장된 URDF 에서 읽는다. 길이가 파라미터인 이상 주석은
자기 위의 값과 어긋날 수 없기 때문이다.

팔 링크에 콜라이더가 아예 없어 벽을 통과했다. 박스로 넣었다.

임포터는 robot/vica_arm 이 있으면 옆에 vica_arm_1 을 만들고 아무도 안 읽는
줄에만 그렇게 말했다. 스테이지는 옛 자산을 계속 참조하므로 방금 늘린 팔이 옛
길이로 렌더되고 아무것도 이상해 보이지 않는다. 이제 옛 것을 .prev 로 옮긴다 —
지우지 않는 이유는, 교체할 export 가 이미 실패한 줄 모르고 지웠다가 자산을
없앤 적이 있기 때문이다.

replay_render 에 --exposure 를 넣었다. 실내는 지붕이 키 라이트를 막고 닫힌
천장이 돔도 대부분 막아서, 뷰포트에서 멀쩡한 방이 두 스톱 어둡게 렌더된다.
오피스가 정전난 것처럼 나왔다. 무대를 밝히면 병원이 틀어지므로 카메라에서
올린다.

drive_scripted 에 --origin-yaw 를 넣었다. --origin 과 같은 문제인데 출발점이
안 움직여서 더 놓치기 쉽다. /odom 은 스폰 방향을 0 이라고 부르므로, 105도로
스폰한 로봇의 기록은 무대의 x 축을 따라 달린 것으로 남는다. 오피스 주행은
로비로 갔는데 렌더는 창문 쪽으로 다시 그렸다.

Co-Authored-By: Claude Opus 5 (1M context) <noreply@anthropic.com>
Claude-Session: https://claude.ai/code/session_015N9GDZdxWCMXWPookPuWGD

File: src/vica_description/urdf/VICA.xacro (robot description, xacro)
@@ -86,9 +86,29 @@
      mass at the top of the robot is what the forward tipping margin pays for,
      and scripts/mass_properties.py prints that.
-     So the design number to try is arm_link3_len:=0.30 arm_link4_len:=0.28,
-     and it is a flag rather than an edit because it is not what ROBOTIS
-     sells. -->
-<xacro:arg name="arm_link3_len" default="0.128" />
-<xacro:arg name="arm_link4_len" default="0.124" />
+     So 0.30 / 0.28 is the design, and it is now the default. The arm as
+     ROBOTIS sells it is still one flag away, arm_link3_len:=0.128
+     arm_link4_len:=0.124, and that is the pair to quote whenever a number
+     has to match their catalogue.
+     What the extra length costs is the motor, not the tipping margin. Every
+     joint is an XM430-W350-T, 4.1 N.m of stall torque at 12 V, and joint2
+     carries the whole arm at whatever distance it is held out. Held straight
+     out, stock, scripts/arm_torque.py reads 1.15 N.m of arm and 2.16 more for
+     a 500 g payload: 81% of stall, already a pose to pass through rather than
+     hold. At 0.30 / 0.28 the arm alone is 2.80, which is 68% of stall with
+     nothing in the gripper at all, and the same payload takes it to 6.56, which is
+     half again more than the motor has.
+     So the long arm reaches the button and cannot carry the shopping. That is
+     the right trade for what this arm is for, which is pressing lift buttons
+     and pointing: pressing pushes along the arm and barely loads joint2 at
+     all, and a pose with the elbow folded is a fraction of the straight-out
+     figure. What it does rule out is holding anything at arm's length:
+     handing over a parcel, carrying a tray. That wants a bigger servo at
+     joint2, an XM540-W270 at 7.0 N.m, or a spring across the shoulder to
+     carry the arm's own 2.80. A shorter link is not the answer, because the
+     length is what puts the gripper 151 mm past the robot's nose. scripts/arm_torque.py prints
+     these numbers from the expanded URDF, so they follow the lengths instead
+     of being retyped after them. -->
+<xacro:arg name="arm_link3_len" default="0.30" />
+<xacro:arg name="arm_link4_len" default="0.28" />
 <xacro:arg name="arm_link5_len" default="0.126" />
 <!-- Geometry exported from CAD is expressed in metres through a 0.001 mesh scale.

File: src/vica_description/urdf/omx_arm.xacro (robot description, xacro)
@@ -25,6 +25,9 @@
   Lengthening moves the joints and does not stretch the meshes. A link built
   longer than ROBOTIS sells is our own part, and drawing their casing scaled
-  along one axis would be a picture of something that does not exist. The mesh
-  sits at the joint and the extra length shows as the gap to the next one.
+  along one axis would be a picture of something that does not exist. So the
+  casing is drawn at its own size and the length we added is drawn as what it
+  will be: a plain machined bar from the end of their casing to the next
+  joint. Leaving that bar out is what made the first long render look like an
+  arm coming apart, with the far half floating free of the near half.
   Lengthening
   ~~~~~~~~~~~
@@ -55,16 +58,31 @@
     <xacro:property name="m4_stock" value="0.132745620" />
     <xacro:property name="m5_stock" value="0.143275730" />
-    <xacro:property name="m3" value="${m3_stock * link3_len / l3_stock}" />
-    <xacro:property name="m4" value="${m4_stock * link4_len / l4_stock}" />
-    <xacro:property name="m5" value="${m5_stock * link5_len / l5_stock}" />
-    <!-- XM430-W350-T: 1.5 N.m stall at 12 V, 46 RPM no-load. Effort is given
-         as the stall figure and velocity as 46 RPM in rad/s. Neither is read
-         by the driving stack; they are here so a motion planner cannot ask
-         for something the servo could not do. -->
+    <!-- A lengthened link weighs its own casing plus the bar we add, and not
+         a scaled copy of the casing. Scaling the whole mass with length was
+         the first model here and it is wrong in the expensive direction: most
+         of ROBOTIS's 138 g is the bracket that carries the servo at each end,
+         and brackets do not get longer. It overstated the long arm's shoulder
+         torque by about 15%.
+         0.60 kg/m is a 30 by 30 mm aluminium tube with a 2 mm wall, which is
+         the section the `ext` box below is drawn at. -->
+    <xacro:property name="bar_kg_per_m" value="0.60" />
+    <xacro:property name="m3" value="${m3_stock + bar_kg_per_m * (link3_len - l3_stock)}" />
+    <xacro:property name="m4" value="${m4_stock + bar_kg_per_m * (link4_len - l4_stock)}" />
+    <xacro:property name="m5" value="${m5_stock + bar_kg_per_m * (link5_len - l5_stock)}" />
+    <!-- XM430-W350-T. The servo stalls at 4.1 N.m at 12 V and runs 46 RPM
+         with nothing on it; the 1.5 here is the working limit ROBOTIS puts in
+         their own URDF, which is the number a planner should be held to and
+         is well under stall on purpose. Velocity is that 46 RPM in rad/s.
+         Neither is read by the driving stack. scripts/arm_torque.py compares
+         what a pose asks of joint2 against the stall figure. -->
     <xacro:property name="joint_effort" value="1.5" />
     <xacro:property name="joint_velocity" value="4.82" />
-    <!-- The arm's own section, for the box stand-ins. -->
+    <!-- The arm's own section, for the box stand-ins. `ext` is the bar that
+         fills the length we added: slimmer than the casing, because that is
+         what a machined extension between two DYNAMIXEL brackets looks like
+         and because drawing it flush with the casing would hide the join. -->
     <xacro:property name="w" value="0.045" />
-    <xacro:macro name="omx_link" params="name mass seg axis:=z mesh:=''">
+    <xacro:property name="ext" value="0.030" />
+    <xacro:macro name="omx_link" params="name mass seg axis:=z mesh:='' stock:=0">
       <link name="${name}">
         <visual>
@@ -86,4 +104,32 @@
           </xacro:unless>
         </visual>
+        <!-- The part we make. Only appears when the link is longer than the
+             one ROBOTIS sells, which is why the stock arm still renders as
+             exactly their arm. stock=0 is how a link says it never lengthens:
+             without that test link1 and link2 came out with a bar drawn over
+             the whole of their casing, because everything is longer than
+             nothing. -->
+        <xacro:if value="${mesh != '' and stock > 0 and seg > stock + 0.001}">
+          <visual>
+            <origin xyz="${axis == 'x' and (stock + seg)/2 or 0} 0 ${axis == 'z' and (stock + seg)/2 or 0}"
+                    rpy="0 0 0"/>
+            <geometry>
+              <box size="${axis == 'x' and (seg - stock) or ext} ${ext} ${axis == 'z' and (seg - stock) or ext}"/>
+            </geometry>
+            <material name="silver"/>
+          </visual>
+        </xacro:if>
+        <!-- Collision is a box over the whole link and never the mesh. A
+             collider is what the solver spends its time on, and a triangle
+             soup per link on a moving arm is the expensive way to learn that.
+             Without any collider at all the arm passes through walls, which
+             is worse than an approximate one. -->
+        <collision>
+          <origin xyz="${axis == 'x' and seg/2 or 0} 0 ${axis == 'z' and seg/2 or 0}"
+                  rpy="0 0 0"/>
+          <geometry>
+            <box size="${axis == 'x' and seg or w} ${w} ${axis == 'z' and seg or w}"/>
+          </geometry>
+        </collision>
         <inertial>
           <origin xyz="${axis == 'x' and seg/2 or 0} 0 ${axis == 'z' and seg/2 or 0}"
@@ -117,5 +163,5 @@
              effort="${joint_effort}" velocity="${joint_velocity}"/>
     </joint>
-    <xacro:omx_link name="${prefix}link3" mass="${m3}" mesh="link3" seg="${link3_len}" axis="z"/>
+    <xacro:omx_link name="${prefix}link3" mass="${m3}" mesh="link3" seg="${link3_len}" axis="z" stock="${l3_stock}"/>
     <joint name="${prefix}joint2" type="revolute">
       <origin xyz="0.0 0.0 0.0595" rpy="0 0 0"/>
@@ -126,5 +172,5 @@
              effort="${joint_effort}" velocity="${joint_velocity}"/>
     </joint>
-    <xacro:omx_link name="${prefix}link4" mass="${m4}" mesh="link4" seg="${link4_len}" axis="x"/>
+    <xacro:omx_link name="${prefix}link4" mass="${m4}" mesh="link4" seg="${link4_len}" axis="x" stock="${l4_stock}"/>
     <joint name="${prefix}joint3" type="revolute">
       <!-- 0.024 of forward offset is ROBOTIS's; the vertical part is the
@@ -137,5 +183,5 @@
              effort="${joint_effort}" velocity="${joint_velocity}"/>
     </joint>
-    <xacro:omx_link name="${prefix}link5" mass="${m5}" mesh="link5" seg="${link5_len}" axis="x"/>
+    <xacro:omx_link name="${prefix}link5" mass="${m5}" mesh="link5" seg="${link5_len}" axis="x" stock="${l5_stock}"/>
     <joint name="${prefix}joint4" type="revolute">
       <origin xyz="${link4_len} 0.0 0.0" rpy="0 0 0"/>

File: src/vica_description/urdf/vica_arm.urdf (robot description, URDF)
Before this commit: robot VICA, 25 links, 24 joints
Links:
- link omx_link1: geometry collision box size=0.045 0.045 0.034; visual mesh filename=package://vica_description/meshes/omx/link1.stl scale=0.001 0.001 0.001
- link omx_link2: geometry collision box size=0.045 0.045 0.0595; visual mesh filename=package://vica_description/meshes/omx/link2.stl scale=0.001 0.001 0.001
- link omx_link3: mass 0.13850917 -> 0.24170916999999997; geometry collision box size=0.045 0.045 0.3; visual box size=0.03 0.03 0.172
- link omx_link4: mass 0.13274562 -> 0.22634562000000003; geometry collision box size=0.28 0.045 0.045; visual box size=0.15600000000000003 0.03 0.03
- link omx_link5: geometry collision box size=0.126 0.045 0.045; visual mesh filename=package://vica_description/meshes/omx/link5.stl scale=0.001 0.001 0.001
Joints:
- joint omx_joint3: origin xyz=0.024 0 0.128 rpy=0 0 0 -> xyz=0.024 0 0.3 rpy=0 0 0
- joint omx_joint4: origin xyz=0.124 0.0 0.0 rpy=0 0 0 -> xyz=0.28 0.0 0.0 rpy=0 0 0
